File: design/sensors_dev/_saved_eval_sensors.sch (KiCad schematic (older format))
At the start: 34 parts, among them J4 Conn_01x12, U2 BMC150, U3 LSM6DS3HTR, U4 FXAS21002, U5 MS5607-02BA03, U6 LIS3DHTR

Commit message: Add footprints and decoupling caps to some ICs
Parts:
- U3: footprint Package_LGA:Bosch_LGA-14_3x2.5mm_P0.5mm -> LSM6DS3:PQFN50P300X250X86-14N
- U5: footprint (none) -> MS560702BA03-50:SON125P300X500X100-8N
- U6: footprint (none) -> LIS3DHTR:LGA16R50P5X3_300X300X100N
Changed lines of the file:
@@
 F 0 "U6" H 2650 6650 60  0000 C CNN
 F 1 "LIS3DHTR" H 3350 5700 60  0000 C CNN
-F 2 "" H 2950 6100 60  0001 C CNN
+F 2 "LIS3DHTR:LGA16R50P5X3_300X300X100N" H 2950 6100 60  0001 C CNN
 F 3 "" H 2950 6100 60  0001 C CNN
 	1    2950 6100
@@
 F 0 "U3" H 6150 3100 60  0000 C CNN
 F 1 "LSM6DS3HTR" H 7000 2100 60  0000 C CNN
-F 2 "Package_LGA:Bosch_LGA-14_3x2.5mm_P0.5mm" H 6450 2400 60  0001 C CNN
+F 2 "LSM6DS3:PQFN50P300X250X86-14N" H 6450 2400 60  0001 C CNN
 F 3 "" H 6450 2400 60  0001 C CNN
 	1    6550 2650
@@
 F 0 "U5" H 5850 6000 60  0000 C CNN
 F 1 "MS5607-02BA03" H 6100 5450 60  0000 C CNN
-F 2 "" H 6100 5450 60  0001 C CNN
+F 2 "MS560702BA03-50:SON125P300X500X100-8N" H 6100 5450 60  0001 C CNN
 F 3 "" H 6100 5450 60  0001 C CNN
 	1    6050 5450
